Commit message: Update CMakeList % file path in .xacro

File: ouster_description/urdf/os1_32.urdf.xacro (robot description, xacro)
@@ -37,8 +37,8 @@
       </collision>
       <visual name="lidar_visual">
-        <origin xyz="0 0 0.3" rpy="0 0 0"/>
+        <origin xyz="0 0 0" rpy="0 0 0"/>
         <geometry>
           <!-- <mesh filename="$(find ouster_description)/meshes/${file_visual}.stl" /> -->
-          <mesh filename="$(find ouster_description)/meshes/${file_visual}.dae" />
+          <mesh filename="file://$(find ouster_description)/meshes/${file_visual}.dae" />
         </geometry>
       </visual>

File: ouster_description/urdf/os1_64.urdf.xacro (robot description, xacro)
@@ -40,5 +40,5 @@
         <geometry>
           <!-- <mesh filename="$(find ouster_description)/meshes/${file_visual}.stl" /> -->
-          <mesh filename="$(find ouster_description)/meshes/${file_visual}.dae" />
+          <mesh filename="file://$(find ouster_description)/meshes/${file_visual}.dae" />
         </geometry>
       </visual>

Commit message: add gpu option

File: ouster_description/urdf/os1_32.urdf.xacro (robot description, xacro)
@@ -53,61 +53,91 @@
     </joint>
     <gazebo reference="${name}_lidar">
-      <sensor type="${gpu_str}ray" name="${name}_lidar">
-        <pose>0 0 0 0 0 0</pose>
-        <visualize>false</visualize>
-        <update_rate>${hz}</update_rate>
-        <ray>
-          <scan>
-            <vertical>
-              <samples>32</samples>
-              <resolution>1</resolution>
-              <min_angle>${min_angle_v*PI/180.0}</min_angle>
-              <max_angle>${max_angle_v*PI/180.0}</max_angle>
-            </vertical>
-            <horizontal>
-              <samples>${samples}</samples>
-              <resolution>1</resolution>
-              <min_angle>-${PI}</min_angle>
-              <max_angle>${PI}</max_angle>
-            </horizontal>
-          </scan>
-          <range>
-            <min>${min_range}</min>
-            <max>${max_range}</max>
-            <resolution>0.03</resolution>
-          </range>
-          <noise>
-            <type>gaussian</type>
-            <mean>0.0</mean>
-            <stddev>0.000000000001</stddev>
-          </noise>
-        </ray>
-        <plugin name="gazebo_ros_laser_controller" filename="libgazebo_ros_ouster_${gpu_str}laser.so">
-            <ros>
-              <namespace>/${name}</namespace>
-              <remapping>~/out:=${prefix}/points</remapping>
-            </ros>
-          <!-- <topicName>${prefix}/points</topicName> -->
-          <frameName>${name}_lidar</frameName>
-          <min_range>${min_range}</min_range>
-          <max_range>${max_range}</max_range>
-          <gaussianNoise>${noise}</gaussianNoise>
-        </plugin>
-      </sensor>
+      <xacro:if value="${gpu}">
+        <sensor type="${gpu_str}ray" name="${name}_lidar">
+          <pose>0 0 0 0 0 0</pose>
+          <visualize>false</visualize>
+          <update_rate>${hz}</update_rate>
+          <ray>
+            <scan>
+              <vertical>
+                <samples>32</samples>
+                <resolution>1</resolution>
+                <min_angle>${min_angle_v*PI/180.0}</min_angle>
+                <max_angle>${max_angle_v*PI/180.0}</max_angle>
+              </vertical>
+              <horizontal>
+                <samples>${samples}</samples>
+                <resolution>1</resolution>
+                <min_angle>-${PI}</min_angle>
+                <max_angle>${PI}</max_angle>
+              </horizontal>
+            </scan>
+            <range>
+              <min>${min_range}</min>
+              <max>${max_range}</max>
+              <resolution>0.03</resolution>
+            </range>
+            <noise>
+              <type>gaussian</type>
+              <mean>0.0</mean>
+              <stddev>0.000000000001</stddev>
+            </noise>
+          </ray>
+          <plugin name="gazebo_ros_laser_controller" filename="libgazebo_ros_ouster_laser.so">
+              <ros>
+                <namespace>/${name}</namespace>
+                <remapping>~/out:=${prefix}/points</remapping>
+              </ros>
+            <frameName>${name}_lidar</frameName>
+            <min_range>${min_range}</min_range>
+            <max_range>${max_range}</max_range>
+            <gaussianNoise>${noise}</gaussianNoise>
+          </plugin>
+        </sensor>
+      </xacro:if>
+      <xacro:unless value="${gpu}">
+        <sensor type="ray" name="${name}_lidar">
+          <pose>0 0 0 0 0 0</pose>
+          <visualize>false</visualize>
+          <update_rate>${hz}</update_rate>
+          <ray>
+            <scan>
+              <vertical>
+                <samples>32</samples>
+                <resolution>1</resolution>
+                <min_angle>${min_angle_v*PI/180.0}</min_angle>
+                <max_angle>${max_angle_v*PI/180.0}</max_angle>
+              </vertical>
+              <horizontal>
+                <samples>${samples}</samples>
+                <resolution>1</resolution>
+                <min_angle>-${PI}</min_angle>
+                <max_angle>${PI}</max_angle>
+              </horizontal>
+            </scan>
+            <range>
+              <min>${min_range}</min>
+              <max>${max_range}</max>
+              <resolution>0.03</resolution>
+            </range>
+            <noise>
+              <type>gaussian</type>
+              <mean>0.0</mean>
+              <stddev>0.000000000001</stddev>
+            </noise>
+          </ray>
+          <plugin name="gazebo_ros_laser_controller" filename="libgazebo_ros_ouster_laser.so">
+              <ros>
+                <namespace>/${name}</namespace>
+                <remapping>~/out:=${prefix}/points</remapping>
+              </ros>
+            <frameName>${name}_lidar</frameName>
+            <min_range>${min_range}</min_range>
+            <max_range>${max_range}</max_range>
+            <gaussianNoise>${noise}</gaussianNoise>
+          </plugin>
+        </sensor>
+      </xacro:unless>
     </gazebo>
-    <!-- <link name="${name}_imu"/>
-    <joint name="${name}_imu_joint" type="fixed">
-      <parent link="${name}_sensor"/>
-      <child link="${name}_imu"/>
-    </joint> -->
-    <!-- <gazebo reference="${name}_imu">
-      <sensor type="imu" name="${name}_imu_sensor">
-        <pose>0 0 0 0 0 0</pose>
-        <always_on>true</always_on>
-        <update_rate>100</update_rate>
-        <visualize>true</visualize>
-        <topic>${prefix}/imu</topic>
-      </sensor>
-    </gazebo> -->
   </xacro:macro>
 </robot>

File: ouster_description/urdf/os1_32_example.urdf.xacro (robot description, xacro)
@@ -31,5 +31,5 @@
   </link>
   <xacro:include filename="$(find ouster_description)/urdf/os1_32.urdf.xacro"/>
-  <xacro:os1_32 parent="base_footprint" name="os" prefix="/ouster" hz="10" samples="512">
+  <xacro:os1_32 parent="base_footprint" name="os" prefix="/ouster" hz="10" samples="512" gpu="${gpu}">
     <origin xyz="0 0 0.4" rpy="0 0 0" />
   </xacro:os1_32>

File: ouster_description/urdf/os1_64.urdf.xacro (robot description, xacro)
@@ -53,61 +53,93 @@
     </joint>
     <gazebo reference="${name}_lidar">
-      <sensor type="${gpu_str}ray" name="${name}_lidar">
-        <pose>0 0 0 0 0 0</pose>
-        <visualize>false</visualize>
-        <update_rate>${hz}</update_rate>
-        <ray>
-          <scan>
-            <vertical>
-              <samples>64</samples>
-              <resolution>1</resolution>
-              <min_angle>${min_angle_v*PI/180.0}</min_angle>
-              <max_angle>${max_angle_v*PI/180.0}</max_angle>
-            </vertical>
-            <horizontal>
-              <samples>${samples}</samples>
-              <resolution>1</resolution>
-              <min_angle>-${PI}</min_angle>
-              <max_angle>${PI}</max_angle>
-            </horizontal>
-          </scan>
-          <range>
-            <min>${min_range}</min>
-            <max>${max_range}</max>
-            <resolution>0.03</resolution>
-          </range>
-          <noise>
-            <type>gaussian</type>
-            <mean>0.0</mean>
-            <stddev>0.000000000001</stddev>
-          </noise>
-        </ray>
-        <plugin name="gazebo_ros_laser_controller" filename="libgazebo_ros_ouster_${gpu_str}laser.so">
-            <ros>
-              <namespace>/${name}</namespace>
-              <remapping>~/out:=${prefix}/points</remapping>
-            </ros>
-          <!-- <topicName>${prefix}/points</topicName> -->
-          <frameName>${name}_lidar</frameName>
-          <min_range>${min_range}</min_range>
-          <max_range>${max_range}</max_range>
-          <gaussianNoise>${noise}</gaussianNoise>
-        </plugin>
-      </sensor>
+      <xacro:if value="${gpu}">
+        <sensor type="${gpu_str}ray" name="${name}_lidar">
+          <pose>0 0 0 0 0 0</pose>
+          <visualize>false</visualize>
+          <update_rate>${hz}</update_rate>
+          <ray>
+            <scan>
+              <vertical>
+                <samples>64</samples>
+                <resolution>1</resolution>
+                <min_angle>${min_angle_v*PI/180.0}</min_angle>
+                <max_angle>${max_angle_v*PI/180.0}</max_angle>
+              </vertical>
+              <horizontal>
+                <samples>${samples}</samples>
+                <resolution>1</resolution>
+                <min_angle>-${PI}</min_angle>
+                <max_angle>${PI}</max_angle>
+              </horizontal>
+            </scan>
+            <range>
+              <min>${min_range}</min>
+              <max>${max_range}</max>
+              <resolution>0.03</resolution>
+            </range>
+            <noise>
+              <type>gaussian</type>
+              <mean>0.0</mean>
+              <stddev>0.000000000001</stddev>
+            </noise>
+          </ray>
+          <plugin name="gazebo_ros_laser_controller" filename="libgazebo_ros_ouster_laser.so">
+              <ros>
+                <namespace>/${name}</namespace>
+                <remapping>~/out:=${prefix}/points</remapping>
+              </ros>
+            <!-- <topicName>${prefix}/points</topicName> -->
+            <frameName>${name}_lidar</frameName>
+            <min_range>${min_range}</min_range>
+            <max_range>${max_range}</max_range>
+            <gaussianNoise>${noise}</gaussianNoise>
+          </plugin>
+        </sensor>
+      </xacro:if>
+      <xacro:unless value="${gpu}">
+        <sensor type="ray" name="${name}_lidar">
+          <pose>0 0 0 0 0 0</pose>
+          <visualize>false</visualize>
+          <update_rate>${hz}</update_rate>
+          <ray>
+            <scan>
+              <vertical>
+                <samples>64</samples>
+                <resolution>1</resolution>
+                <min_angle>${min_angle_v*PI/180.0}</min_angle>
+                <max_angle>${max_angle_v*PI/180.0}</max_angle>
+              </vertical>
+              <horizontal>
+                <samples>${samples}</samples>
+                <resolution>1</resolution>
+                <min_angle>-${PI}</min_angle>
+                <max_angle>${PI}</max_angle>
+              </horizontal>
+            </scan>
+            <range>
+              <min>${min_range}</min>
+              <max>${max_range}</max>
+              <resolution>0.03</resolution>
+            </range>
+            <noise>
+              <type>gaussian</type>
+              <mean>0.0</mean>
+              <stddev>0.000000000001</stddev>
+            </noise>
+          </ray>
+          <plugin name="gazebo_ros_laser_controller" filename="libgazebo_ros_ouster_laser.so">
+              <ros>
+                <namespace>/${name}</namespace>
+                <remapping>~/out:=${prefix}/points</remapping>
+              </ros>
+            <!-- <topicName>${prefix}/points</topicName> -->
+            <frameName>${name}_lidar</frameName>
+            <min_range>${min_range}</min_range>
+            <max_range>${max_range}</max_range>
+            <gaussianNoise>${noise}</gaussianNoise>
+          </plugin>
+        </sensor>
+      </xacro:unless>
     </gazebo>
-    <!-- <link name="${name}_imu"/>
-    <joint name="${name}_imu_joint" type="fixed">
-      <parent link="${name}_sensor"/>
-      <child link="${name}_imu"/>
-    </joint> -->
-    <!-- <gazebo reference="${name}_imu">
-      <sensor type="imu" name="${name}_imu_sensor">
-        <pose>0 0 0 0 0 0</pose>
-        <always_on>true</always_on>
-        <update_rate>100</update_rate>
-        <visualize>true</visualize>
-        <topic>${prefix}/imu</topic>
-      </sensor>
-    </gazebo> -->
   </xacro:macro>
 </robot>

File: ouster_description/urdf/os1_64_example.urdf.xacro (robot description, xacro)
@@ -31,5 +31,5 @@
   </link>
   <xacro:include filename="$(find ouster_description)/urdf/os1_64.urdf.xacro"/>
-  <xacro:os1_64 parent="base_footprint" name="os" prefix="/ouster" hz="10" samples="512">
+  <xacro:os1_64 parent="base_footprint" name="os" prefix="/ouster" hz="10" samples="512" gpu="${gpu}">
     <origin xyz="0 0 0.4" rpy="0 0 0" />
   </xacro:os1_64>
